File: cz18_badge.kicad_pcb (KiCad board)
At the start: 2 copper layers, 100 x 100 mm, 16 parts, among them U1 NRF24L01_Breakout

Commit message: Added todo comments
Other:
- board text added: "TODO: - Finalise PCB design concept - Layout components - Create VCC and GND planes on front and back of the badge - Route traces"
Changed lines of the file:
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@@
     (area 49.924999 29.924999 150.075001 130.075001)
     (thickness 1.6)
-    (drawings 4)
+    (drawings 5)
     (tracks 0)
     (zones 0)
@@
     )
   )
+  (gr_text "TODO:\n\n- Finalise PCB design concept\n- Layout components\n- Create VCC and GND planes on front and back of the badge\n- Route traces" (at 186 53) (layer F.Cu)
+    (effects (font (size 1.5 1.5) (thickness 0.3)) (justify left))
+  )
   (gr_line (start 50 130) (end 50 30) (angle 90) (layer Edge.Cuts) (width 0.15))
